Commit message: fix

File: rosrider_description/urdf/next.urdf (robot description, URDF)
Before this commit: robot next, 8 links, 7 joints
Joints:
- joint scan_joint: origin xyz=-0.062 0 0.0706 rpy=0 0 0 -> xyz=-0.166 0 0.0706 rpy=0 0 0

Commit message: urdf first

File: rosrider_description/urdf/next.urdf (robot description, URDF)
Before this commit: robot next, 8 links, 7 joints
Joints:
- joint battery_joint: origin xyz=-0.08383 0 0.0116 rpy=0 0 0 -> xyz=-0.06883 0 0.0116 rpy=0 0 0
- joint caster_back_joint: origin xyz=-0.14835 0 -0.02425 rpy=0 0 0 -> xyz=-0.178 0 -0.02425 rpy=0 0 0
- joint scan_joint: origin xyz=-0.166 0 0.0706 rpy=0 0 0 -> xyz=-0.166 -0.006 0.0706 rpy=0 0 0

Commit message: imu fixed

File: rosrider_description/urdf/next.urdf (robot description, URDF)
Before this commit: robot next, 8 links, 7 joints
Links:
- removed link wheel_left_link
- removed link wheel_right_link
- link imu_link: geometry visual mesh filename=package://rosrider_description/meshes/fximu3e.dae scale=1 1 1
Joints:
- removed joint wheel_left_joint
- removed joint wheel_right_joint
- joint imu_joint: origin xyz=0.0 0.0 0.0656 rpy=0 0 0 -> xyz=0.041 0.0 0.0496 rpy=0 0 0

Commit message: joints uncommented

File: rosrider_description/urdf/next.urdf (robot description, URDF)
Before this commit: robot next, 6 links, 5 joints
Links:
- added link wheel_left_link; visual mesh filename=package://rosrider_description/meshes/wheel_left.dae scale=1 1 1
- added link wheel_right_link; visual mesh filename=package://rosrider_description/meshes/wheel_right.dae scale=1 1 1
Joints:
- added joint wheel_left_joint: type continuous, parent base_link, child wheel_left_link, origin xyz=0.0 0.0896 0.0 rpy=-1.57 0 0, axis 0 0 1
- added joint wheel_right_joint: type continuous, parent base_link, child wheel_right_link, origin xyz=0.0 -0.0896 0.0 rpy=-1.57 0 0, axis 0 0 1

Commit message: stls added

File: rosrider_description/urdf/next.urdf (robot description, URDF)
Before this commit: robot next, 8 links, 7 joints
Links:
- link base_link: geometry visual mesh filename=package://rosrider_description/meshes/next_urdf.dae scale=1 1 1

Commit message: echo

File: rosrider_description/urdf/next.urdf (robot description, URDF)
Before this commit: robot next, 8 links, 7 joints
Joints:
- joint battery_joint: origin xyz=-0.06883 0 0.0116 rpy=0 0 0 -> xyz=-0.07183 0 0.0116 rpy=0 0 0
- joint caster_back_joint: origin xyz=-0.178 0 -0.02425 rpy=0 0 0 -> xyz=-0.1842 0 -0.02425 rpy=0 0 0
- joint imu_joint: origin xyz=0.041 0.0 0.0496 rpy=0 0 0 -> xyz=0.0378 0.0 0.0473 rpy=0 0 0
- joint scan_joint: origin xyz=-0.166 -0.006 0.0706 rpy=0 0 0 -> xyz=-0.1692 0.0 0.061 rpy=0 0 0
- joint wheel_left_joint: origin xyz=0.0 0.0896 0.0 rpy=-1.57 0 0 -> xyz=0.0 0.087 0.0 rpy=-1.57 0 0
- joint wheel_right_joint: origin xyz=0.0 -0.0896 0.0 rpy=-1.57 0 0 -> xyz=0.0 -0.087 0.0 rpy=-1.57 0 0

Commit message: barb

File: rosrider_description/urdf/next.urdf (robot description, URDF)
Before this commit: robot next, 8 links, 7 joints
Links:
- link caster_back_link: geometry visual mesh filename=package://rosrider_description/meshes/vac_wheel.dae scale=1 1 1
Joints:
- joint battery_joint: origin xyz=-0.06883 0 0.0116 rpy=0 0 0 -> xyz=-0.07183 0 0.0116 rpy=0 0 0
- joint caster_back_joint: origin xyz=-0.178 0 -0.02425 rpy=0 0 0 -> xyz=-0.2002 0 -0.02425 rpy=0 0 0
- joint imu_joint: origin xyz=0.041 0.0 0.0496 rpy=0 0 0 -> xyz=0.0378 0.0 0.0473 rpy=0 0 0
- joint scan_joint: origin xyz=-0.166 -0.006 0.0706 rpy=0 0 0 -> xyz=-0.1692 0.0 0.061 rpy=0 0 0
- joint wheel_left_joint: origin xyz=0.0 0.0896 0.0 rpy=-1.57 0 0 -> xyz=0.0 0.087 0.0 rpy=-1.57 0 0
- joint wheel_right_joint: origin xyz=0.0 -0.0896 0.0 rpy=-1.57 0 0 -> xyz=0.0 -0.087 0.0 rpy=-1.57 0 0

Commit message: to robot next

File: rosrider_description/urdf/next.urdf (robot description, URDF)
Before this commit: robot next, 8 links, 7 joints
Links:
- removed link caster_back_link
- added link wheel_castor_link; collision mesh filename=package://rosrider_description/meshes/vac_wheel.stl scale=0.001 0.001 0.001; visual mesh filename=package://rosrider_description/meshes/vac_wheel.dae scale=1 1 1
- added link wheel_steering_link
Joints:
- removed joint caster_back_joint
- added joint wheel_castor_joint: type continuous, parent wheel_steering_link, child wheel_castor_link, origin xyz=-0.016 0 -0.01275 rpy=0 0 0, axis 0 1 0
- added joint wheel_steering_joint: type continuous, parent base_link, child wheel_steering_link, origin xyz=-0.1842 0 -0.00875 rpy=0 0 0, axis 0 0 1

Commit message: new version

File: rosrider_description/urdf/next.urdf (robot description, URDF)
Before this commit: robot next, 9 links, 8 joints
Joints:
- joint scan_joint: origin xyz=-0.1692 0.0 0.061 rpy=0 0 0 -> xyz=-0.1692 0.0 0.06125 rpy=0 0 0
