Commit message: optical frame

File: rosrider_description/urdf/sorcerer.urdf (robot description, URDF)
Before this commit: robot sorcerer, 8 links, 7 joints
Links:
- added link camera_link; visual mesh filename=package://rosrider_description/meshes/cam_stand.dae scale=1 1 1
- added link camera_optical_frame
Joints:
- added joint camera_joint: type fixed, parent base_link, child camera_link, origin xyz=0.05615 0.0 0.04928 rpy=0 0 0
- added joint optical_joint: type fixed, parent camera_link, child camera_optical_frame, origin xyz=0.0032 0.0 0.02762 rpy=0 0.3071 0

Commit message: optical frame tilt1

File: rosrider_description/urdf/sorcerer.urdf (robot description, URDF)
Before this commit: robot sorcerer, 10 links, 9 joints
Joints:
- joint optical_joint: origin xyz=0.0032 0.0 0.02762 rpy=0 0.3071 0 -> xyz=0.0032 0.0 0.02762 rpy=-0.3072 0.0 -1.5708

Commit message: optical frame tilt3

File: rosrider_description/urdf/sorcerer.urdf (robot description, URDF)
Before this commit: robot sorcerer, 10 links, 9 joints
Joints:
- joint optical_joint: origin xyz=0.0032 0.0 0.02762 rpy=-0.3072 0.0 -1.5708 -> xyz=0.0032 0.0 0.02762 rpy=-0.3072 -1.5708 -1.5708

Commit message: tags

File: rosrider_description/urdf/sorcerer.urdf (robot description, URDF)
Before this commit: robot sorcerer, 10 links, 9 joints
Joints:
- joint optical_joint: origin xyz=0.0032 0.0 0.02762 rpy=-0.3072 -1.5708 -1.5708 -> xyz=0.0032 0.0 0.02762 rpy=-1.87 0.0 -1.57

Commit message: st

File: rosrider_description/urdf/sorcerer.urdf (robot description, URDF)
Before this commit: robot sorcerer, 10 links, 9 joints
Joints:
- joint optical_joint: origin xyz=0.0032 0.0 0.02762 rpy=-1.87 0.0 -1.57 -> xyz=0.0032 0.0 0.02762 rpy=-1.57 0.0 -1.57

Commit message: st2

File: rosrider_description/urdf/sorcerer.urdf (robot description, URDF)
Before this commit: robot sorcerer, 10 links, 9 joints
Joints:
- joint optical_joint: origin xyz=0.0032 0.0 0.02762 rpy=-1.57 0.0 -1.57 -> xyz=0.0032 0.0 0.02762 rpy=-1.97 0.0 -1.57

Commit message: st3

File: rosrider_description/urdf/sorcerer.urdf (robot description, URDF)
Before this commit: robot sorcerer, 10 links, 9 joints
Joints:
- joint optical_joint: origin xyz=0.0032 0.0 0.02762 rpy=-1.97 0.0 -1.57 -> xyz=0.0032 0.0 0.02762 rpy=-1.87 0.0 -1.57
