Commit message: refactor0

File: rosrider_description/urdf/caretta.urdf (robot description, URDF)
Before this commit: robot sorcerer, 10 links, 9 joints
Links:
- removed link camera_link
- removed link camera_optical_frame
- removed link caster_back_link
- added link wheel_castor_link; visual mesh filename=package://rosrider_description/meshes/vac_wheel.dae scale=1 1 1
- added link wheel_steering_link
- link base_link: geometry visual mesh filename=package://rosrider_description/meshes/caretta.dae scale=1 1 1
- link battery_link: geometry visual box size=0.0736 0.1535 0.0276
- link imu_link: geometry visual mesh filename=package://rosrider_description/meshes/fximu3e.dae scale=1 1 1
Joints:
- removed joint camera_joint
- removed joint caster_back_joint
- removed joint optical_joint
- added joint wheel_castor_joint: type continuous, parent wheel_steering_link, child wheel_castor_link, origin xyz=-0.016 0 -0.01275 rpy=0 0 0, axis 0 1 0
- added joint wheel_steering_joint: type continuous, parent base_link, child wheel_steering_link, origin xyz=-0.1842 0 -0.00875 rpy=0 0 0, axis 0 0 1
- joint battery_joint: origin xyz=-0.034057 0 0.057282 rpy=0 0 0 -> xyz=-0.07183 0 0.0116 rpy=0 0 0
- joint imu_joint: origin xyz=0.008 0 0.0739 rpy=0 0 0 -> xyz=0.0378 0.0 0.0473 rpy=0 0 0
- joint scan_joint: origin xyz=-0.067 0 0.0989 rpy=0 0 0 -> xyz=-0.1692 0.0 0.06125 rpy=0 0 0
- joint wheel_left_joint: origin xyz=0.0 0.05 0.0 rpy=-1.57 0 0 -> xyz=0.0 0.087 0.0 rpy=-1.57 0 0
- joint wheel_right_joint: origin xyz=0.0 -0.05 0.0 rpy=-1.57 0 0 -> xyz=0.0 -0.087 0.0 rpy=-1.57 0 0

File: rosrider_description/urdf/duckiebot.urdf (robot description, URDF)
Before this commit: robot next, 9 links, 8 joints
Links:
- removed link base_scan
- added link camera_optical_frame; visual mesh filename=package://rosrider_description/meshes/cam_stand_optical.dae scale=1 1 1
- link base_link: geometry visual mesh filename=package://rosrider_description/meshes/duckiebot.dae scale=1 1 1
- link battery_link: geometry visual box size=0.1368 0.0639 0.016
- link imu_link: geometry visual mesh filename=package://rosrider_description/meshes/fximu.dae scale=1 1 1
- link wheel_castor_link: geometry visual sphere radius=0.01
Joints:
- removed joint scan_joint
- added joint camera_joint: type fixed, parent base_link, child camera_optical_frame, origin xyz=0.05935 0.0 0.07690 rpy=-1.87 0.0 -1.57
- joint battery_joint: origin xyz=-0.07183 0 0.0116 rpy=0 0 0 -> xyz=-0.034057 0 0.057282 rpy=0 0 0
- joint imu_joint: origin xyz=0.0378 0.0 0.0473 rpy=0 0 0 -> xyz=0.008 0 0.0739 rpy=0 0 0
- joint wheel_castor_joint: origin xyz=-0.016 0 -0.01275 rpy=0 0 0 -> xyz=0 0 0 rpy=0 0 0
- joint wheel_left_joint: origin xyz=0.0 0.087 0.0 rpy=-1.57 0 0 -> xyz=0.0 0.05 0.0 rpy=-1.57 0 0
- joint wheel_right_joint: origin xyz=0.0 -0.087 0.0 rpy=-1.57 0 0 -> xyz=0.0 -0.05 0.0 rpy=-1.57 0 0
- joint wheel_steering_joint: origin xyz=-0.1842 0 -0.00875 rpy=0 0 0 -> xyz=-0.09 0 -0.02425 rpy=0 0 0

Commit message: REFACTOR 1

File: rosrider_description/urdf/caretta.urdf (robot description, URDF)
Before this commit: robot caretta, 9 links, 8 joints
Joints:
- joint wheel_castor_joint: type continuous -> fixed
- joint wheel_steering_joint: type continuous -> fixed

Commit message: refactor 3

File: rosrider_description/urdf/caretta.urdf (robot description, URDF)
Before this commit: robot caretta, 9 links, 8 joints
Links:
- link base_link: geometry visual mesh filename=package://rosrider_description/meshes/caretta2.dae scale=1 1 1

File: rosrider_description/urdf/caretta_gz.urdf (robot description, URDF)
Before this commit: robot duckiebot, 9 links, 8 joints
Links:
- removed link camera_optical_frame
- added link base_scan; visual mesh filename=package://rosrider_description/meshes/ldlidar.dae scale=1 1 1
- link base_link: geometry visual mesh filename=package://rosrider_description/meshes/caretta_body.dae scale=1 1 1
- link battery_link: geometry visual box size=0.0736 0.1535 0.0276
- link imu_link: geometry visual mesh filename=package://rosrider_description/meshes/fximu3e.dae scale=1 1 1
- link wheel_castor_link: geometry visual mesh filename=package://rosrider_description/meshes/vac_wheel.dae scale=1 1 1
Joints:
- removed joint camera_joint
- added joint scan_joint: type fixed, parent base_link, child base_scan, origin xyz=-0.1692 0.0 0.06125 rpy=0 0 0
- joint battery_joint: origin xyz=-0.034057 0 0.057282 rpy=0 0 0 -> xyz=-0.07183 0 0.0116 rpy=0 0 0
- joint imu_joint: origin xyz=0.008 0 0.0739 rpy=0 0 0 -> xyz=0.0378 0.0 0.0473 rpy=0 0 0
- joint wheel_castor_joint: origin xyz=0 0 0 rpy=0 0 0 -> xyz=-0.016 0 -0.01275 rpy=0 0 0
- joint wheel_left_joint: origin xyz=0.0 0.05 0.0 rpy=-1.57 0 0 -> xyz=0.0 0.087 0.0 rpy=-1.57 0 0
- joint wheel_right_joint: origin xyz=0.0 -0.05 0.0 rpy=-1.57 0 0 -> xyz=0.0 -0.087 0.0 rpy=-1.57 0 0
- joint wheel_steering_joint: origin xyz=-0.09 0 -0.02425 rpy=0 0 0 -> xyz=-0.1842 0 -0.00875 rpy=0 0 0

Commit message: refactor 3a

File: rosrider_description/urdf/caretta.urdf (robot description, URDF)
Before this commit: robot caretta, 9 links, 8 joints
Links:
- link base_link: geometry visual mesh filename=package://rosrider_description/meshes/caretta_body.dae scale=1 1 1

Commit message: S

File: rosrider_description/urdf/caretta.urdf (robot description, URDF)
Before this commit: robot caretta, 9 links, 8 joints
Joints:
- joint wheel_castor_joint: type fixed -> continuous
- joint wheel_left_joint: axis 0 0 1 -> 0 1 0; origin xyz=0.0 0.087 0.0 rpy=-1.57 0 0 -> xyz=0.0 0.087 0.0 rpy=0 0 0
- joint wheel_right_joint: axis 0 0 1 -> 0 1 0; origin xyz=0.0 -0.087 0.0 rpy=-1.57 0 0 -> xyz=0.0 -0.087 0.0 rpy=0 0 0
- joint wheel_steering_joint: type fixed -> continuous

File: rosrider_description/urdf/duckiebot.urdf (robot description, URDF)
Before this commit: robot duckiebot, 9 links, 8 joints
Links:
- removed link wheel_steering_link
- link imu_link: geometry visual mesh filename=package://rosrider_description/meshes/fximu3e.dae scale=1 1 1
Joints:
- removed joint wheel_steering_joint
- joint camera_joint: origin xyz=0.05935 0.0 0.07690 rpy=-1.87 0.0 -1.57 -> xyz=0.05935 0.0 0.07690 rpy=-1.87 0.0 -1.570796
- joint imu_joint: origin xyz=0.008 0 0.0739 rpy=0 0 0 -> xyz=0 0 0.0739 rpy=0 0 0
- joint wheel_castor_joint: axis 0 1 0 -> (none); origin xyz=0 0 0 rpy=0 0 0 -> xyz=-0.095 0 -0.02425 rpy=0 0 0; parent wheel_steering_link -> base_link
- joint wheel_left_joint: axis 0 0 1 -> 0 1 0; origin xyz=0.0 0.05 0.0 rpy=-1.57 0 0 -> xyz=0.0 0.05 0.0 rpy=0 0 0
- joint wheel_right_joint: axis 0 0 1 -> 0 1 0; origin xyz=0.0 -0.05 0.0 rpy=-1.57 0 0 -> xyz=0.0 -0.05 0.0 rpy=0 0 0
