Commit message: MID

File: rosrider_description/urdf/beagle.urdf (robot description, URDF)
Before this commit: robot beagle, 11 links, 10 joints
Links:
- removed link base_scan
- added link base_scan_3d; visual box size=0.02 0.1 0.02
Joints:
- joint scan_joint: child base_scan -> base_scan_3d; origin xyz=0.0925 0.0 0.085 rpy=0 0 0 -> xyz=0.1025 0.0 0.1 rpy=0 0 0

File: rosrider_description/urdf/beagle_front.urdf (robot description, URDF)
Before this commit: robot beagle_front, 10 links, 9 joints
Links:
- removed link imu1_link
- removed link imu_link
Joints:
- removed joint imu1_joint
- removed joint imu_joint

File: rosrider_description/urdf/caterpillar.urdf (robot description, URDF)
Before this commit: robot caterpillar, 15 links, 14 joints
Links:
- removed link imu1_link
- removed link imu_link
Joints:
- removed joint imu1_joint
- removed joint imu_joint

File: rosrider_description/urdf/rover.urdf (robot description, URDF)
Before this commit: robot rover, 7 links, 6 joints
Links:
- added link base_scan_3d; visual box size=0.02 0.1 0.02
Joints:
- added joint scan_joint: type fixed, parent base_link, child base_scan_3d, origin xyz=0.01 0.0 0.34 rpy=0 0 0

Commit message: T1

File: rosrider_description/urdf/beagle.urdf (robot description, URDF)
Before this commit: robot beagle, 11 links, 10 joints
Links:
- removed link base_footprint
- removed link imu1_link
Joints:
- removed joint base_joint
- removed joint imu1_joint
- joint imu_joint: origin xyz=0.16 0 0 rpy=0 0 0 -> xyz=0.14 0 0 rpy=0 0 0
- joint scan_joint: origin xyz=0.1025 0.0 0.1 rpy=0 0 0 -> xyz=0 0 0.1 rpy=0 0 0

File: rosrider_description/urdf/beagle_front.urdf (robot description, URDF)
Before this commit: robot beagle_front, 8 links, 7 joints
Links:
- removed link base_footprint
- added link base_scan_3d; visual box size=0.02 0.1 0.02
- added link imu_link; visual mesh filename=package://rosrider_description/meshes/fximu3e.dae scale=1 1 1
Joints:
- removed joint base_joint
- added joint imu_joint: type fixed, parent front_link, child imu_link, origin xyz=0.085 0 0 rpy=0 0 0
- added joint scan_joint: type fixed, parent front_link, child base_scan_3d, origin xyz=0 0.0 0.1 rpy=0 0 0

File: rosrider_description/urdf/caretta.urdf (robot description, URDF)
Before this commit: robot caretta, 9 links, 8 joints
Joints:
- joint base_joint: origin xyz=0.0 0.0 0.03425 rpy=0 0 0 -> xyz=0 0 0.03425 rpy=0 0 0

File: rosrider_description/urdf/caterpillar.urdf (robot description, URDF)
Before this commit: robot caterpillar, 13 links, 12 joints
Links:
- removed link base_footprint
- added link base_scan_3d; visual box size=0.02 0.1 0.02
- added link imu_link; visual mesh filename=package://rosrider_description/meshes/fximu3e.dae scale=1 1 1
Joints:
- removed joint base_joint
- added joint imu_joint: type fixed, parent front_link, child imu_link, origin xyz=0.105 0 0 rpy=0 0 0
- added joint scan_joint: type fixed, parent front_link, child base_scan_3d, origin xyz=0 0 0.1 rpy=0 0 0

File: rosrider_description/urdf/rover.urdf (robot description, URDF)
Before this commit: robot rover, 8 links, 7 joints
Joints:
- joint scan_joint: origin xyz=0.01 0.0 0.34 rpy=0 0 0 -> xyz=0 0.0 0.34 rpy=0 0 0
